File: Project Files/Kicad/Achroma_Choc/Achroma_Choc.kicad_pcb (KiCad board)
At the start: 2 copper layers, 116.6 x 99.4 mm, 78 parts, among them SW1 RESET, SW2 SW_SPDT_312, U2 nice_nano

Commit message: updated project files
Parts:
- removed the G*** at (65.2, 84.3)
- moved G*** 1.36 mm to (82.9, 71.7)
